Commit message: added cell description, gripper node and moveit wrapper

File: src/kuka_eki/kuka_common/urdf/kuka.ros2_control.xacro (robot description, xacro)
@@ -1,5 +1,5 @@
 <?xml version="1.0"?>
 <robot xmlns:xacro="http://www.ros.org/wiki/xacro">
-    <xacro:macro name="kuka_ros2_control" params="name robot_prefix initial_positions_file robot_ip robot_port use_fake_hardware">
+    <xacro:macro name="kuka_ros2_control" params="name robot_prefix initial_positions_file robot_ip eki_robot_port use_fake_hardware">
         <xacro:property name="initial_positions" value="${load_yaml(initial_positions_file)['initial_positions']}"/>
         <ros2_control name="${name}" type="system">
@@ -11,5 +11,5 @@
                     <plugin>kuka_eki_hw_interface/KukaEkiHardwareInterface</plugin>
                     <param name="robot_ip">${robot_ip}</param>
-                    <param name="robot_port">${robot_port}</param>
+                    <param name="eki_robot_port">${eki_robot_port}</param>
                 </xacro:unless>
             </hardware>

File: src/kuka_eki/kuka_kr10_description/urdf/kr10r1100sixx.xacro (robot description, xacro)
@@ -4,8 +4,8 @@
     <xacro:arg name="initial_positions_file" default="$(find kuka_common)/config/initial_positions.yaml"/>
     <xacro:arg name="robot_ip" default="10.181.116.41"/>
-    <xacro:arg name="robot_port" default="54600"/>
+    <xacro:arg name="eki_robot_port" default="54600"/>
     <xacro:arg name="use_fake_hardware" default="true"/>
     <xacro:kuka_kr10r1100sixx prefix="" initial_positions_file="$(arg initial_positions_file)"
-                              robot_ip="$(arg robot_ip)" robot_port="$(arg robot_port)"
+                              robot_ip="$(arg robot_ip)" eki_robot_port="$(arg eki_robot_port)"
                               use_fake_hardware="$(arg use_fake_hardware)"/>
 </robot>

File: src/kuka_eki/kuka_kr10_description/urdf/kr10r1100sixx_macro.xacro (robot description, xacro)
@@ -4,5 +4,5 @@
     <xacro:include filename="$(find kuka_common)/urdf/common_materials.xacro"/>
     <xacro:include filename="$(find kuka_common)/urdf/kuka.ros2_control.xacro"/>
-    <xacro:macro name="kuka_kr10r1100sixx" params="prefix initial_positions_file robot_ip robot_port use_fake_hardware">
+    <xacro:macro name="kuka_kr10r1100sixx" params="prefix initial_positions_file robot_ip eki_robot_port use_fake_hardware">
         <link name="${prefix}base_link">
             <visual>
@@ -175,5 +175,5 @@
         <xacro:kuka_ros2_control name="kuka_control" robot_prefix="${prefix}"
                                  initial_positions_file="${initial_positions_file}"
-                                 robot_ip="${robot_ip}" robot_port="${robot_port}"
+                                 robot_ip="${robot_ip}" eki_robot_port="${eki_robot_port}"
                                  use_fake_hardware="${use_fake_hardware}"/>
     </xacro:macro>

File: src/kuka_eki/kuka_kr10_description/urdf/kr10r900_2.xacro (robot description, xacro)
@@ -4,8 +4,8 @@
     <xacro:arg name="initial_positions_file" default="$(find kuka_common)/config/initial_positions.yaml"/>
     <xacro:arg name="robot_ip" default="10.181.116.41"/>
-    <xacro:arg name="robot_port" default="54600"/>
+    <xacro:arg name="eki_robot_port" default="54600"/>
     <xacro:arg name="use_fake_hardware" default="true"/>
     <xacro:kuka_kr10r900_2 prefix="" initial_positions_file="$(arg initial_positions_file)"
-                           robot_ip="$(arg robot_ip)" robot_port="$(arg robot_port)"
+                           robot_ip="$(arg robot_ip)" eki_robot_port="$(arg eki_robot_port)"
                            use_fake_hardware="$(arg use_fake_hardware)"/>
 </robot>

File: src/kuka_eki/kuka_kr10_description/urdf/kr10r900_2_macro.xacro (robot description, xacro)
@@ -3,5 +3,5 @@
     <xacro:include filename="$(find kuka_common)/urdf/common_materials.xacro"/>
     <xacro:include filename="$(find kuka_common)/urdf/kuka.ros2_control.xacro"/>
-    <xacro:macro name="kuka_kr10r900_2" params="prefix initial_positions_file robot_ip robot_port use_fake_hardware">
+    <xacro:macro name="kuka_kr10r900_2" params="prefix initial_positions_file robot_ip eki_robot_port use_fake_hardware">
         <link name="${prefix}base_link">
             <visual>
@@ -175,5 +175,5 @@
         <xacro:kuka_ros2_control name="kuka_control" robot_prefix="${prefix}"
                                  initial_positions_file="${initial_positions_file}"
-                                 robot_ip="${robot_ip}" robot_port="${robot_port}"
+                                 robot_ip="${robot_ip}" eki_robot_port="${eki_robot_port}"
                                  use_fake_hardware="${use_fake_hardware}"/>
     </xacro:macro>

File: src/kuka_eki/kuka_kr120_description/urdf/kr120r2500pro_macro.xacro (robot description, xacro)
@@ -2,5 +2,5 @@
 <robot xmlns:xacro="http://wiki.ros.org/xacro">
     <xacro:include filename="$(find kuka_common)/urdf/kuka.ros2_control.xacro"/>
-    <xacro:macro name="kuka_kr120r2500pro" params="prefix initial_positions_file robot_ip robot_port use_fake_hardware">
+    <xacro:macro name="kuka_kr120r2500pro" params="prefix initial_positions_file robot_ip eki_robot_port use_fake_hardware">
         <!-- LINKS -->
         <!-- base link -->
@@ -219,5 +219,5 @@
         <xacro:kuka_ros2_control name="kuka_control" robot_prefix="${prefix}"
                                  initial_positions_file="${initial_positions_file}"
-                                 robot_ip="${robot_ip}" robot_port="${robot_port}"
+                                 robot_ip="${robot_ip}" eki_robot_port="${eki_robot_port}"
                                  use_fake_hardware="${use_fake_hardware}"/>
     </xacro:macro>

File: src/kuka_eki/kuka_kr120_description/urdf/robot.urdf.xacro (robot description, xacro)
@@ -5,8 +5,8 @@
     <xacro:arg name="initial_positions_file" default="$(find kuka_common)/config/initial_positions.yaml"/>
     <xacro:arg name="robot_ip" default="10.181.116.41"/>
-    <xacro:arg name="robot_port" default="54600"/>
+    <xacro:arg name="eki_robot_port" default="54600"/>
     <xacro:arg name="use_fake_hardware" default="true"/>
     <xacro:kuka_kr120r2500pro prefix="" initial_positions_file="$(arg initial_positions_file)"
-                              robot_ip="$(arg robot_ip)" robot_port="$(arg robot_port)"
+                              robot_ip="$(arg robot_ip)" eki_robot_port="$(arg eki_robot_port)"
                               use_fake_hardware="$(arg use_fake_hardware)"/>
 </robot>

File: src/kuka_eki/kuka_kr150_description/urdf/kr150_2_macro.xacro (robot description, xacro)
@@ -2,5 +2,5 @@
 <robot xmlns:xacro="http://wiki.ros.org/xacro">
     <xacro:include filename="$(find kuka_common)/urdf/kuka.ros2_control.xacro"/>
-    <xacro:macro name="kuka_kr150_2" params="prefix initial_positions_file robot_ip robot_port use_fake_hardware">
+    <xacro:macro name="kuka_kr150_2" params="prefix initial_positions_file robot_ip eki_robot_port use_fake_hardware">
         <!-- LINKS -->
         <!-- base link -->
@@ -185,5 +185,5 @@
         <xacro:kuka_ros2_control name="kuka_control" robot_prefix="${prefix}"
                                  initial_positions_file="${initial_positions_file}"
-                                 robot_ip="${robot_ip}" robot_port="${robot_port}"
+                                 robot_ip="${robot_ip}" eki_robot_port="${eki_robot_port}"
                                  use_fake_hardware="${use_fake_hardware}"/>
     </xacro:macro>

File: src/kuka_eki/kuka_kr150_description/urdf/robot.urdf.xacro (robot description, xacro)
@@ -4,8 +4,8 @@
     <xacro:arg name="initial_positions_file" default="$(find kuka_common)/config/initial_positions.yaml"/>
     <xacro:arg name="robot_ip" default="10.181.116.41"/>
-    <xacro:arg name="robot_port" default="54600"/>
+    <xacro:arg name="eki_robot_port" default="54600"/>
     <xacro:arg name="use_fake_hardware" default="true"/>
     <xacro:kuka_kr150_2 prefix="" initial_positions_file="$(arg initial_positions_file)"
-                        robot_ip="$(arg robot_ip)" robot_port="$(arg robot_port)"
+                        robot_ip="$(arg robot_ip)" eki_robot_port="$(arg eki_robot_port)"
                         use_fake_hardware="$(arg use_fake_hardware)"/>
 </robot>

File: src/kuka_eki/kuka_kr16_description/urdf/kr16_2_macro.xacro (robot description, xacro)
@@ -2,5 +2,5 @@
 <robot xmlns:xacro="http://wiki.ros.org/xacro">
     <xacro:include filename="$(find kuka_common)/urdf/kuka.ros2_control.xacro"/>
-    <xacro:macro name="kuka_kr16_2" params="prefix initial_positions_file robot_ip robot_port use_fake_hardware">
+    <xacro:macro name="kuka_kr16_2" params="prefix initial_positions_file robot_ip eki_robot_port use_fake_hardware">
         <!-- LINKS -->
         <!-- base link -->
@@ -220,5 +220,5 @@
         <xacro:kuka_ros2_control name="kuka_control" robot_prefix="${prefix}"
                                  initial_positions_file="${initial_positions_file}"
-                                 robot_ip="${robot_ip}" robot_port="${robot_port}"
+                                 robot_ip="${robot_ip}" eki_robot_port="${eki_robot_port}"
                                  use_fake_hardware="${use_fake_hardware}"/>
     </xacro:macro>

File: src/kuka_eki/kuka_kr16_description/urdf/robot.urdf.xacro (robot description, xacro)
@@ -5,8 +5,8 @@
     <xacro:arg name="initial_positions_file" default="$(find kuka_common)/config/initial_positions.yaml"/>
     <xacro:arg name="robot_ip" default="10.181.116.41"/>
-    <xacro:arg name="robot_port" default="54600"/>
+    <xacro:arg name="eki_robot_port" default="54600"/>
     <xacro:arg name="use_fake_hardware" default="true"/>
     <xacro:kuka_kr16_2 prefix="" initial_positions_file="$(arg initial_positions_file)"
-                       robot_ip="$(arg robot_ip)" robot_port="$(arg robot_port)"
+                       robot_ip="$(arg robot_ip)" eki_robot_port="$(arg eki_robot_port)"
                        use_fake_hardware="$(arg use_fake_hardware)"/>
 </robot>

File: src/kuka_eki/kuka_kr210_description/urdf/kr210l150_macro.xacro (robot description, xacro)
@@ -2,5 +2,5 @@
 <robot xmlns:xacro="http://wiki.ros.org/xacro">
     <xacro:include filename="$(find kuka_common)/urdf/kuka.ros2_control.xacro"/>
-    <xacro:macro name="kuka_kr210l150" params="prefix initial_positions_file robot_ip robot_port use_fake_hardware">
+    <xacro:macro name="kuka_kr210l150" params="prefix initial_positions_file robot_ip eki_robot_port use_fake_hardware">
         <!-- links -->
         <link name="${prefix}base_link">
@@ -232,5 +232,5 @@
         <xacro:kuka_ros2_control name="kuka_control" robot_prefix="${prefix}"
                                  initial_positions_file="${initial_positions_file}"
-                                 robot_ip="${robot_ip}" robot_port="${robot_port}"
+                                 robot_ip="${robot_ip}" eki_robot_port="${eki_robot_port}"
                                  use_fake_hardware="${use_fake_hardware}"/>
     </xacro:macro>

File: src/kuka_eki/kuka_kr210_description/urdf/robot.urdf.xacro (robot description, xacro)
@@ -4,8 +4,8 @@
     <xacro:arg name="initial_positions_file" default="$(find kuka_common)/config/initial_positions.yaml"/>
     <xacro:arg name="robot_ip" default="10.181.116.41"/>
-    <xacro:arg name="robot_port" default="54600"/>
+    <xacro:arg name="eki_robot_port" default="54600"/>
     <xacro:arg name="use_fake_hardware" default="true"/>
     <xacro:kuka_kr210l150 prefix="" initial_positions_file="$(arg initial_positions_file)"
-                          robot_ip="$(arg robot_ip)" robot_port="$(arg robot_port)"
+                          robot_ip="$(arg robot_ip)" eki_robot_port="$(arg eki_robot_port)"
                           use_fake_hardware="$(arg use_fake_hardware)"/>
 </robot>

File: src/kuka_eki/kuka_kr3_description/urdf/kr3r540_macro.xacro (robot description, xacro)
@@ -3,5 +3,5 @@
     <xacro:include filename="$(find kuka_common)/urdf/common_materials.xacro"/>
     <xacro:include filename="$(find kuka_common)/urdf/kuka.ros2_control.xacro"/>
-    <xacro:macro name="kuka_kr3r540" params="prefix initial_positions_file robot_ip robot_port use_fake_hardware">
+    <xacro:macro name="kuka_kr3r540" params="prefix initial_positions_file robot_ip eki_robot_port use_fake_hardware">
         <link name="${prefix}base_link">
             <visual>
@@ -173,5 +173,5 @@
         <xacro:kuka_ros2_control name="kuka_control" robot_prefix="${prefix}"
                                  initial_positions_file="${initial_positions_file}"
-                                 robot_ip="${robot_ip}" robot_port="${robot_port}"
+                                 robot_ip="${robot_ip}" eki_robot_port="${eki_robot_port}"
                                  use_fake_hardware="${use_fake_hardware}"/>
     </xacro:macro>

File: src/kuka_eki/kuka_kr3_description/urdf/robot.urdf.xacro (robot description, xacro)
@@ -4,8 +4,8 @@
     <xacro:arg name="initial_positions_file" default="$(find kuka_common)/config/initial_positions.yaml"/>
     <xacro:arg name="robot_ip" default="10.181.116.41"/>
-    <xacro:arg name="robot_port" default="54600"/>
+    <xacro:arg name="eki_robot_port" default="54600"/>
     <xacro:arg name="use_fake_hardware" default="true"/>
     <xacro:kuka_kr3r540 prefix="" initial_positions_file="$(arg initial_positions_file)"
-                        robot_ip="$(arg robot_ip)" robot_port="$(arg robot_port)"
+                        robot_ip="$(arg robot_ip)" eki_robot_port="$(arg eki_robot_port)"
                         use_fake_hardware="$(arg use_fake_hardware)"/>
 </robot>

File: src/kuka_eki/kuka_kr5_description/urdf/kr5_arc_macro.xacro (robot description, xacro)
@@ -2,5 +2,5 @@
 <robot xmlns:xacro="http://wiki.ros.org/xacro">
     <xacro:include filename="$(find kuka_common)/urdf/kuka.ros2_control.xacro"/>
-    <xacro:macro name="kuka_kr5_arc" params="prefix initial_positions_file robot_ip robot_port use_fake_hardware">
+    <xacro:macro name="kuka_kr5_arc" params="prefix initial_positions_file robot_ip eki_robot_port use_fake_hardware">
         <!-- LINKS -->
         <!-- base link -->
@@ -281,5 +281,5 @@
         <xacro:kuka_ros2_control name="kuka_control" robot_prefix="${prefix}"
                                  initial_positions_file="${initial_positions_file}"
-                                 robot_ip="${robot_ip}" robot_port="${robot_port}"
+                                 robot_ip="${robot_ip}" eki_robot_port="${eki_robot_port}"
                                  use_fake_hardware="${use_fake_hardware}"/>
     </xacro:macro>

File: src/kuka_eki/kuka_kr5_description/urdf/robot.urdf.xacro (robot description, xacro)
@@ -4,8 +4,8 @@
     <xacro:arg name="initial_positions_file" default="$(find kuka_common)/config/initial_positions.yaml"/>
     <xacro:arg name="robot_ip" default="10.181.116.41"/>
-    <xacro:arg name="robot_port" default="54600"/>
+    <xacro:arg name="eki_robot_port" default="54600"/>
     <xacro:arg name="use_fake_hardware" default="true"/>
     <xacro:kuka_kr5_arc prefix="" initial_positions_file="$(arg initial_positions_file)"
-                        robot_ip="$(arg robot_ip)" robot_port="$(arg robot_port)"
+                        robot_ip="$(arg robot_ip)" eki_robot_port="$(arg eki_robot_port)"
                         use_fake_hardware="$(arg use_fake_hardware)"/>
 </robot>

File: src/kuka_eki/kuka_kr6_description/urdf/kr6r700sixx.xacro (robot description, xacro)
@@ -4,8 +4,8 @@
     <xacro:arg name="initial_positions_file" default="$(find kuka_common)/config/initial_positions.yaml"/>
     <xacro:arg name="robot_ip" default="10.181.116.41"/>
-    <xacro:arg name="robot_port" default="54600"/>
+    <xacro:arg name="eki_robot_port" default="54600"/>
     <xacro:arg name="use_fake_hardware" default="true"/>
     <xacro:kuka_kr6r700sixx prefix="" initial_positions_file="$(arg initial_positions_file)"
-                            robot_ip="$(arg robot_ip)" robot_port="$(arg robot_port)"
+                            robot_ip="$(arg robot_ip)" eki_robot_port="$(arg eki_robot_port)"
                             use_fake_hardware="$(arg use_fake_hardware)"/>
 </robot>

File: src/kuka_eki/kuka_kr6_description/urdf/kr6r700sixx_macro.xacro (robot description, xacro)
@@ -4,5 +4,5 @@
     <xacro:include filename="$(find kuka_common)/urdf/common_materials.xacro"/>
     <xacro:include filename="$(find kuka_common)/urdf/kuka.ros2_control.xacro"/>
-    <xacro:macro name="kuka_kr6r700sixx" params="prefix initial_positions_file robot_ip robot_port use_fake_hardware">
+    <xacro:macro name="kuka_kr6r700sixx" params="prefix initial_positions_file robot_ip eki_robot_port use_fake_hardware">
         <link name="${prefix}base_link">
             <visual>
@@ -175,5 +175,5 @@
         <xacro:kuka_ros2_control name="kuka_control" robot_prefix="${prefix}"
                                  initial_positions_file="${initial_positions_file}"
-                                 robot_ip="${robot_ip}" robot_port="${robot_port}"
+                                 robot_ip="${robot_ip}" eki_robot_port="${eki_robot_port}"
                                  use_fake_hardware="${use_fake_hardware}"/>
     </xacro:macro>

File: src/kuka_eki/kuka_kr6_description/urdf/kr6r900_2.xacro (robot description, xacro)
@@ -4,8 +4,8 @@
     <xacro:arg name="initial_positions_file" default="$(find kuka_common)/config/initial_positions.yaml"/>
     <xacro:arg name="robot_ip" default="10.181.116.41"/>
-    <xacro:arg name="robot_port" default="54600"/>
+    <xacro:arg name="eki_robot_port" default="54600"/>
     <xacro:arg name="use_fake_hardware" default="true"/>
     <xacro:kuka_kr6r900_2 prefix="" initial_positions_file="$(arg initial_positions_file)"
-                          robot_ip="$(arg robot_ip)" robot_port="$(arg robot_port)"
+                          robot_ip="$(arg robot_ip)" eki_robot_port="$(arg eki_robot_port)"
                           use_fake_hardware="$(arg use_fake_hardware)"/>
 </robot>
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