Commit message: upgrade to humble

File: kuka_common/urdf/kuka.ros2_control.xacro (robot description, xacro)
@@ -1,10 +1,12 @@
 <?xml version="1.0"?>
 <robot xmlns:xacro="http://www.ros.org/wiki/xacro">
-    <xacro:macro name="kuka_ros2_control" params="name robot_prefix initial_positions_file robot_ip eki_robot_port use_fake_hardware">
-        <xacro:property name="initial_positions" value="${load_yaml(initial_positions_file)['initial_positions']}"/>
+    <xacro:macro name="kuka_ros2_control"
+                 params="name robot_prefix initial_positions_file robot_ip eki_robot_port use_fake_hardware">
+        <xacro:property name="initial_positions"
+                        value="${xacro.load_yaml(initial_positions_file)['initial_positions']}"/>
         <ros2_control name="${name}" type="system">
             <hardware>
                 <xacro:if value="${use_fake_hardware}">
-                    <plugin>fake_components/GenericSystem</plugin>
+                    <plugin>mock_components/GenericSystem</plugin>
                 </xacro:if>
                 <xacro:unless value="${use_fake_hardware}">
@@ -15,32 +17,38 @@
             </hardware>
             <joint name="${robot_prefix}joint_a1">
-                <param name="initial_position">${initial_positions['joint_a1']}</param>
                 <command_interface name="position"/>
-                <state_interface name="position"/>
+                <state_interface name="position">
+                    <param name="initial_value">${initial_positions['joint_a1']}</param>
+                </state_interface>
             </joint>
             <joint name="${robot_prefix}joint_a2">
-                <param name="initial_position">${initial_positions['joint_a2']}</param>
                 <command_interface name="position"/>
-                <state_interface name="position"/>
+                <state_interface name="position">
+                    <param name="initial_value">${initial_positions['joint_a2']}</param>
+                </state_interface>
             </joint>
             <joint name="${robot_prefix}joint_a3">
-                <param name="initial_position">${initial_positions['joint_a3']}</param>
                 <command_interface name="position"/>
-                <state_interface name="position"/>
+                <state_interface name="position">
+                    <param name="initial_value">${initial_positions['joint_a3']}</param>
+                </state_interface>
             </joint>
             <joint name="${robot_prefix}joint_a4">
-                <param name="initial_position">${initial_positions['joint_a4']}</param>
                 <command_interface name="position"/>
-                <state_interface name="position"/>
+                <state_interface name="position">
+                    <param name="initial_value">${initial_positions['joint_a4']}</param>
+                </state_interface>
             </joint>
             <joint name="${robot_prefix}joint_a5">
-                <param name="initial_position">${initial_positions['joint_a5']}</param>
                 <command_interface name="position"/>
-                <state_interface name="position"/>
+                <state_interface name="position">
+                    <param name="initial_value">${initial_positions['joint_a5']}</param>
+                </state_interface>
             </joint>
             <joint name="${robot_prefix}joint_a6">
-                <param name="initial_position">${initial_positions['joint_a6']}</param>
                 <command_interface name="position"/>
-                <state_interface name="position"/>
+                <state_interface name="position">
+                    <param name="initial_value">${initial_positions['joint_a6']}</param>
+                </state_interface>
             </joint>
         </ros2_control>
